Commit message: faet:urdf文件增加关节限制

File: src/biped_s4/urdf/biped_s4.urdf (robot description, URDF)
Before this commit: robot biped_s4, 61 links, 60 joints
Joints:
- joint l_arm_pitch: limit (none) -> lower=-3.14159 upper=0.523599 effort=20 velocity=1; type continuous -> revolute
- joint l_arm_roll: limit (none) -> lower=-0.349066 upper=2.0944 effort=20 velocity=1; type continuous -> revolute
- joint l_arm_yaw: limit (none) -> lower=-1.5708 upper=1.5708 effort=20 velocity=1; type continuous -> revolute
- joint l_forearm_pitch: limit (none) -> lower=-1.5708 upper=0 effort=20 velocity=1; type continuous -> revolute
- joint l_hand_pitch: limit (none) -> lower=-1.5708 upper=1.5708 effort=20 velocity=1; type continuous -> revolute
- joint l_hand_roll: limit (none) -> lower=-1.5708 upper=1.5708 effort=20 velocity=1; type continuous -> revolute
- joint l_hand_yaw: limit (none) -> lower=-1.5708 upper=1.5708 effort=20 velocity=1; type continuous -> revolute
- joint r_arm_pitch: limit (none) -> lower=-3.14159 upper=0.523599 effort=20 velocity=1; type continuous -> revolute
- joint r_arm_roll: limit (none) -> lower=-2.0944 upper=0.349066 effort=20 velocity=1; type continuous -> revolute
- joint r_arm_yaw: limit (none) -> lower=-1.5708 upper=1.5708 effort=20 velocity=1; type continuous -> revolute
- joint r_forearm_pitch: limit (none) -> lower=-1.5708 upper=0 effort=20 velocity=1; type continuous -> revolute
- joint r_hand_pitch: limit (none) -> lower=-1.5708 upper=1.5708 effort=20 velocity=1; type continuous -> revolute
- joint r_hand_roll: limit (none) -> lower=-1.5708 upper=1.5708 effort=20 velocity=1; type continuous -> revolute
- joint r_hand_yaw: limit (none) -> lower=-1.5708 upper=1.5708 effort=20 velocity=1; type continuous -> revolute
